File: hardware/MrRoboto.brd (EAGLE design)
At the start: 50.8 x 61 mm, 40 parts, among them IC1 NCP1402, U1 ATmega328, U3 LCD-8x2, Y1 16mhz

Commit message: Breaking out additional pins on PCB
Parts:
- added JP14, JP15: (no value), SparkFun-Connectors:1X05
- moved U$2 20.1 mm to (25.4, 21.6)
- moved JP11 1.27 mm to (8.13, 12.7)
Connections:
- removed net N$12: U1.19
- removed net N$13: U1.22
- net A2: now also JP14.3
- net A3: now also JP15.4
- net A4: now also JP15.2
- net A5: now also JP15.3
- net D10: now also JP14.4
- net D2: now also JP14.2
- net GND: now also JP14.1, JP15.1
- net VCC: now also JP14.5, JP15.5
Routing:
- net A2: track 0.00 -> 44.3 mm, vias 0 -> 1
- net A5: track 0.00 -> 39.0 mm, vias 0 -> 1
- net D2: track 0.00 -> 39.0 mm, vias 0 -> 1
- net A4: track 0.00 -> 38.6 mm, vias 0 -> 1
- net A3: track 0.00 -> 36.2 mm, vias 0 -> 1
- net D10: track 0.00 -> 32.2 mm, vias 0 -> 1
- net A0: track 51.8 -> 36.8 mm
- net VCC: track 150.4 -> 144.3 mm
- net D3: track 25.8 -> 21.1 mm
- net DTR: track 13.3 -> 13.8 mm
Other:
- board text added: "5V"
- board text added: "A2"
- board text added: "A3"
- board text added: "A4"
- board text added: "A5"
- board text added: "D10"
- board text added: "D2"
- board text added: "v13"
- board text removed: "4/6/11"
