File: hardware/MrRoboto.sch (EAGLE design)
At the start: 39 parts, among them IC1 NCP1402, U1 ATmega328, U3 LCD-8x2, Y1 16mhz

Commit message: Breaking out additional pins on PCB
Parts:
- added JP14, JP15: (no value), SparkFun-Connectors:M05PTH
Connections:
- removed net N$12: U1.ADC6
- removed net N$13: U1.ADC7
- net A2: now also JP14.3
- net A3: now also JP15.4
- net A4: now also JP15.2
- net A5: now also JP15.3
- net D10: now also JP14.4
- net D2: now also JP14.2
- net GND: now also JP14.1, JP15.1
- net VCC: now also JP14.5, JP15.5
Other:
- note removed: "* C5 changed from 47uF to 68uF"
- note removed: "* IC1 changed from NCP1400 to NCP1402"
- note removed: "* L1 changed from 22uH to 47uH"
- note removed: "* No changes to PCB design"
- note removed: "v12 Fixes:"
